Commit message: feat: Finalize motor calibration with verified offsets, integrate into firmware, and add new ROS 2 control nodes for keyboard and gait control.

File: spotmicro_ws/src/spotmicro_description/urdf/spotmicroai.urdf.xacro (robot description, xacro)
@@ -181,5 +181,5 @@
         <axis xyz="1 0 0" />
         <origin rpy="0 0 0" xyz="-0.093 -0.036 0" />
-        <limit effort="100.0" lower="-1.0" upper="1.0" velocity="0.7" />
+        <limit effort="100.0" lower="-0.2378" upper="0.2608" velocity="0.7" />
         <dynamics damping="3.0" friction="0.5" />
     </joint>
@@ -189,5 +189,5 @@
         <axis xyz="0 1 0" />
         <origin rpy="0 0 0" xyz="0 -0.052 0" />
-        <limit effort="100.0" lower="-2.17" upper="0.97" velocity="0.5" />
+        <limit effort="100.0" lower="-0.0844" upper="0.5292" velocity="0.5" />
         <dynamics damping="3.0" friction="0.0" />
     </joint>
@@ -202,5 +202,5 @@
         <axis xyz="0 1 0" />
         <origin rpy="0 0 0" xyz="-0.01 0 -0.12" />
-        <limit effort="100.0" lower="-0.1" upper="2.59" velocity="0.5" />
+        <limit effort="100.0" lower="-0.6826" upper="1.0124" velocity="0.5" />
         <dynamics damping="3.0" friction="0.5" />
     </joint>
@@ -305,5 +305,5 @@
         <axis xyz="1 0 0" />
         <origin rpy="0 0 0" xyz="-0.093 0.036 0" />
-        <limit effort="100.0" lower="-1.0" upper="1.0" velocity="0.7" />
+        <limit effort="100.0" lower="-0.5983" upper="0.4449" velocity="0.7" />
         <dynamics damping="3.0" friction="0.5" />
     </joint>
@@ -313,5 +313,5 @@
         <axis xyz="0 1 0" />
         <origin rpy="0 0 0" xyz="0 0.052 0" />
-        <limit effort="100.0" lower="-2.17" upper="0.97" velocity="0.5" />
+        <limit effort="100.0" lower="-0.5752" upper="0.8437" velocity="0.5" />
         <dynamics damping="3.0" friction="0.0" />
     </joint>
@@ -326,5 +326,5 @@
         <axis xyz="0 1 0" />
         <origin rpy="0 0 0" xyz="-0.01 0 -0.12" />
-        <limit effort="100.0" lower="-0.1" upper="2.59" velocity="0.5" />
+        <limit effort="100.0" lower="-0.8360" upper="0.6673" velocity="0.5" />
         <dynamics damping="3.0" friction="0.5" />
     </joint>
@@ -429,5 +429,5 @@
         <axis xyz="1 0 0" />
         <origin rpy="0 0 0" xyz="0.093 -0.036 0" />
-        <limit effort="100.0" lower="-1.0" upper="1.0" velocity="0.7" />
+        <limit effort="100.0" lower="-0.3375" upper="0.1841" velocity="0.7" />
         <dynamics damping="3.0" friction="0.5" />
     </joint>
@@ -437,5 +437,5 @@
         <axis xyz="0 1 0" />
         <origin rpy="0 0 0" xyz="0 -0.052 0" />
-        <limit effort="100.0" lower="-2.17" upper="0.97" velocity="0.5" />
+        <limit effort="100.0" lower="-0.4602" upper="0.7516" velocity="0.5" />
         <dynamics damping="3.0" friction="0.0" />
     </joint>
@@ -450,5 +450,5 @@
         <axis xyz="0 1 0" />
         <origin rpy="0 0 0" xyz="-0.01 0 -0.12" />
-        <limit effort="100.0" lower="-0.1" upper="2.59" velocity="0.5" />
+        <limit effort="100.0" lower="-0.6136" upper="0.8744" velocity="0.5" />
         <dynamics damping="3.0" friction="0.5" />
     </joint>
@@ -553,5 +553,5 @@
         <axis xyz="1 0 0" />
         <origin rpy="0 0 0" xyz="0.093 0.036 0" />
-        <limit effort="100.0" lower="-1.0" upper="1.0" velocity="0.7" />
+        <limit effort="100.0" lower="-0.2301" upper="0.4679" velocity="0.7" />
         <dynamics damping="3.0" friction="0.5" />
     </joint>
@@ -561,5 +561,5 @@
         <axis xyz="0 1 0" />
         <origin rpy="0 0 0" xyz="0 0.052 0" />
-        <limit effort="100.0" lower="-2.17" upper="0.97" velocity="0.5" />
+        <limit effort="100.0" lower="-0.6596" upper="0.5139" velocity="0.5" />
         <dynamics damping="3.0" friction="0.0" />
     </joint>
@@ -574,5 +574,5 @@
         <axis xyz="0 1 0" />
         <origin rpy="0 0 0" xyz="-0.01 0 -0.12" />
-        <limit effort="100.0" lower="-0.1" upper="2.59" velocity="0.5" />
+        <limit effort="100.0" lower="-0.8744" upper="0.6289" velocity="0.5" />
         <dynamics damping="3.0" friction="0.5" />
     </joint>
